File: Impedance_Shield_V3.kicad_sch (KiCad schematic)
At the start: 1 part

Commit message: d
Parts:
- removed U1: ~, symbol AD5933:AD5933
Other:
- added sheet AD5933 (AD5933.kicad_sch)
- added sheet Amplifier (Amplifier.kicad_sch)
- added sheet Clock (Clock.kicad_sch)
Changed lines of the file:
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@@
 	(generator_version "8.0")
 	(paper "A4")
-	(symbol
-		(lib_id "AD5933:AD5933")
-		(at 156.21 62.23 0)
-		(unit 2)
-		(exclude_from_sim no)
-		(in_bom yes)
-		(on_board yes)
-		(dnp no)
+	(sheet
+		(at 140.97 120.65)
+		(size 21.59 26.67)
 		(fields_autoplaced yes)
-		(property "Reference" "U1"
-			(at 161.29 58.4199 0)
+		(stroke
+			(width 0.1524)
+			(type solid)
+		)
+		(fill
+			(color 0 0 0 0.0000)
+		)
+		(property "Sheetname" "Amplifier"
+			(at 140.97 119.9384 0)
+			(effects
+				(font
+					(size 1.27 1.27)
+				)
+				(justify left bottom)
+			)
+		)
+		(property "Sheetfile" "Amplifier.kicad_sch"
+			(at 140.97 147.9046 0)
+			(effects
+				(font
+					(size 1.27 1.27)
+				)
+				(justify left top)
+			)
+		)
+		(instances
+			(project "Impedance_Shield_V3"
+				(path "/de23f470-01e5-4133-bf09-5fbd0a8fd2b2"
+					(page "4")
+				)
+			)
+		)
+	)
+	(sheet
+		(at 101.6 137.16)
+		(size 25.4 13.97)
+		(fields_autoplaced yes)
+		(stroke
+			(width 0.1524)
+			(type solid)
+		)
+		(fill
+			(color 0 0 0 0.0000)
+		)
+		(property "Sheetname" "AD5933"
+			(at 101.6 136.4484 0)
+			(effects
+				(font
+					(size 1.27 1.27)
+				)
+				(justify left bottom)
+			)
+		)
+		(property "Sheetfile" "AD5933.kicad_sch"
+			(at 101.6 151.7146 0)
+			(effects
+				(font
+					(size 1.27 1.27)
+				)
+				(justify left top)
+			)
+		)
+		(pin "SDA" input
+			(at 101.6 140.97 180)
 			(effects
 				(font
@@
 			)
 		)
-		(property "Value" "~"
-			(at 161.29 60.325 0)
+		(pin "SCL" input
+			(at 101.6 143.51 180)
 			(effects
 				(font
@@
 			)
 		)
-		(property "Footprint" ""
-			(at 156.21 62.23 0)
+		(pin "ExtClk" input
+			(at 101.6 148.59 180)
+			(effects
+				(font
+					(size 1.27 1.27)
+				)
+				(justify left)
+			)
+		)
+		(pin "Vin" input
+			(at 127 148.59 0)
+			(effects
+				(font
+					(size 1.27 1.27)
+				)
+				(justify right)
+			)
+		)
+		(pin "Vout" input
+			(at 127 140.97 0)
+			(effects
+				(font
+					(size 1.27 1.27)
+				)
+				(justify right)
+			)
+		)
+		(instances
+			(project "Impedance_Shield_V3"
+				(path "/de23f470-01e5-4133-bf09-5fbd0a8fd2b2"
+					(page "3")
+				)
+			)
+		)
+	)
+	(sheet
+		(at 68.58 137.16)
+		(size 17.78 15.24)
+		(fields_autoplaced yes)
+		(stroke
+			(width 0.1524)
+			(type solid)
+		)
+		(fill
+			(color 0 0 0 0.0000)
+		)
+		(property "Sheetname" "Clock"
+			(at 68.58 136.4484 0)
+			(effects
+				(font
+					(size 1.27 1.27)
+				)
+				(justify left bottom)
+			)
+		)
+		(property "Sheetfile" "Clock.kicad_sch"
+			(at 68.58 152.9846 0)
+			(effects
+				(font
+					(size 1.27 1.27)
+				)
+				(justify left top)
+			)
+		)
+		(property "Field2" ""
+			(at 68.58 137.16 0)
 			(effects
 				(font
@@
 			)
 		)
-		(property "Datasheet" ""
-			(at 156.21 62.23 0)
+		(pin "ExClk" input
+			(at 86.36 144.78 0)
 			(effects
 				(font
 					(size 1.27 1.27)
 				)
-				(hide yes)
+				(justify right)
 			)
 		)
-		(property "Description" ""
-			(at 156.21 62.23 0)
+		(pin "OscSw" input
+			(at 68.58 144.78 180)
 			(effects
 				(font
 					(size 1.27 1.27)
 				)
-				(hide yes)
+				(justify left)
 			)
 		)
-		(pin "11"
-		)
-		(pin "15"
-		)
-		(pin "4"
-		)
-		(pin "6"
-		)
-		(pin "10"
-		)
-		(pin "16"
-		)
-		(pin "13"
-		)
-		(pin "1"
-		)
-		(pin "12"
-		)
-		(pin "3"
-		)
-		(pin "14"
-		)
-		(pin "2"
-		)
-		(pin "5"
-		)
-		(pin "8"
-		)
-		(pin "9"
-		)
 		(instances
-			(project ""
+			(project "Impedance_Shield_V3"
 				(path "/de23f470-01e5-4133-bf09-5fbd0a8fd2b2"
-					(reference "U1")
-					(unit 2)
+					(page "2")
 				)
 			)
-		)
-	)
-	(symbol
-		(lib_id "AD5933:AD5933")
-		(at 119.38 50.8 0)
-		(unit 1)
-		(exclude_from_sim no)
-		(in_bom yes)
-		(on_board yes)
-		(dnp no)
-		(fields_autoplaced yes)
-		(property "Reference" "U1"
-			(at 119.38 45.72 0)
-			(effects
-				(font
-					(size 1.27 1.27)
-				)
-			)
-		)
-		(property "Value" "~"
-			(at 119.38 48.26 0)
-			(effects
-				(font
-					(size 1.27 1.27)
-				)
-			)
-		)
-		(property "Footprint" ""
-			(at 119.38 50.8 0)
-			(effects
-				(font
-					(size 1.27 1.27)
-				)
-				(hide yes)
-			)
-		)
-		(property "Datasheet" ""
-			(at 119.38 50.8 0)
-			(effects
-				(font
-					(size 1.27 1.27)
-				)
-				(hide yes)
-			)
-		)
-		(property "Description" ""
-			(at 119.38 50.8 0)
-			(effects
-				(font
-					(size 1.27 1.27)
-				)
-				(hide yes)
-			)
-		)
-		(pin "11"
-		)
-		(pin "15"
-		)
-		(pin "4"
-		)
-		(pin "6"
-		)
-		(pin "10"
-		)
-		(pin "16"
-		)
-		(pin "13"
-		)
-		(pin "1"
-		)
-		(pin "12"
-		)
-		(pin "3"
-		)
-		(pin "14"
-		)
-		(pin "2"
-		)
-		(pin "5"
-		)
-		(pin "8"
-		)
-		(pin "9"
-		)
-		(instances
-			(project ""
-				(path "/de23f470-01e5-4133-bf09-5fbd0a8fd2b2"
-					(reference "U1")
-					(unit 1)
-				)
-			)
